File: SMEE-DESIGNPROJECT.kicad_sch (KiCad schematic)
At the start: 15 parts, among them J1 Conn_02x03_Odd_Even, U2 LM555xN

Commit message: Reposition PCB components; add title block & PDFs
Connections:
- net +3.3V: no longer J1.2 (Pin_2)
- net Aout: now also J1.1 (Pin_1)
- no-connect marks 1 -> 2
Changed lines of the file:
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@@
 		(at 152.4 53.34)
 	)
+	(no_connect
+		(at 55.88 50.8)
+	)
 	(wire
 		(pts
@@
 	(wire
 		(pts
-			(xy 63.5 50.8) (xy 63.5 48.26)
-		)
-		(stroke
-			(width 0)
-			(type default)
-		)
-	)
-	(wire
-		(pts
 			(xy 68.58 111.76) (xy 68.58 114.3)
 		)
@@
 	(wire
 		(pts
-			(xy 55.88 50.8) (xy 63.5 50.8)
-		)
-		(stroke
-			(width 0)
-			(type default)
-		)
-	)
-	(wire
-		(pts
 			(xy 73.66 165.1) (xy 73.66 167.64)
 		)
@@
 	(wire
 		(pts
-			(xy 33.02 50.8) (xy 41.91 50.8)
+			(xy 33.02 50.8) (xy 43.18 50.8)
 		)
 		(stroke
@@
 					(unit 1)
 				)
-			)
-		)
-	)
-	(symbol
-		(lib_id "power:+3.3V")
-		(at 63.5 48.26 0)
-		(mirror y)
-		(unit 1)
-		(exclude_from_sim no)
-		(in_bom yes)
-		(on_board yes)
-		(dnp no)
-		(property "Reference" "#PWR09"
-			(at 63.5 52.07 0)
-			(effects
-				(font
-					(size 1.27 1.27)
-				)
-				(hide yes)
-			)
-		)
-		(property "Value" "+3.3V"
-			(at 63.5 43.18 0)
-			(effects
-				(font
-					(size 1.27 1.27)
-				)
-			)
-		)
-		(property "Footprint" ""
-			(at 63.5 48.26 0)
-			(effects
-				(font
-					(size 1.27 1.27)
-				)
-				(hide yes)
-			)
-		)
-		(property "Datasheet" ""
-			(at 63.5 48.26 0)
-			(effects
-				(font
-					(size 1.27 1.27)
-				)
-				(hide yes)
-			)
-		)
-		(property "Description" "Power symbol creates a global label with name \"+3.3V\""
-			(at 63.5 48.26 0)
-			(effects
-				(font
-					(size 1.27 1.27)
-				)
-				(hide yes)
-			)
-		)
-		(pin "1"
-		)
-		(instances
-			(project "SMEE-DESIGNPROJECT"
-				(path "/cabf21dc-d7cc-491b-8161-8874ca6c5af3"
-					(reference "#PWR09")
-					(unit 1)
-				)

Commit message: Update PCB layout and backups
Change component value (Value: 330 → 100) and perform extensive PCB layout edits: reroute segments, update zone polygons, net assignments, priorities, teardrop attributes, min_thickness/fill settings, island removal and many UUIDs for F.Cu features. Update related project (.kicad_prl) and schematic (.kicad_sch) files to match layout changes. File-level housekeeping: remove one old backup ZIP and add three new backup ZIP snapshots. These changes correct net/geometry assignments and tidy PCB fill/zone settings.
Parts:
- R4: value 330 -> 100
Changed lines of the file:
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@@
 			)
 		)
-		(property "Value" "330"
+		(property "Value" "100"
 			(at 54.61 129.5399 0)
 			(effects
