File: SMEE-DESIGNPROJECT/SMEE-DESIGNPROJECT.kicad_sch (KiCad schematic)
At the start: 15 parts, among them J1 Conn_01x05, U1 TLC555xP

Commit message: Adjust PCB footprints, traces and copper zones
Modify SMEE-DESIGNPROJECT.kicad_pcb to tweak component placements (small XY adjustments for axial resistor and diode), adjust trace segments (endpoints, added short segments, updated UUIDs), and reorganize copper zones/teardrop pad-via polygons and priorities. Add two backup ZIPs under SMEE-DESIGNPROJECT-backups. Also update project files (.kicad_prl, .kicad_sch). These changes address alignment and copper-pour/connection corrections on the PCB.
Parts:
- C1: value 1n -> 10p
- R5: value 1k -> 220k
Changed lines of the file:
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@@
 			)
 		)
-		(property "Value" "1k"
+		(property "Value" "220k"
 			(at 93.98 109.2199 0)
 			(effects
@@
 			)
 		)
-		(property "Value" "1n"
+		(property "Value" "10p"
 			(at 95.25 121.9199 0)
 			(effects

Commit message: Update KiCad footprints, active layer, and backups
Remove two old backup ZIPs and add two new timestamped backups in SMEE-DESIGNPROJECT/SMEE-DESIGNPROJECT-backups. Change board active_layer from 5 to 0 in SMEE-DESIGNPROJECT.kicad_prl. Update two footprints in SMEE-DESIGNPROJECT.kicad_sch: capacitor pitch changed from P2.50mm to P2.00mm, and diode footprint changed to D_DO-35_SOD27_P10.16mm_Horizontal.
Parts:
- C3: footprint Capacitor_THT:CP_Radial_D5.0mm_P2.50mm -> Capacitor_THT:CP_Radial_D5.0mm_P2.00mm
- D1: footprint Diode_THT:D_A-405_P10.16mm_Horizontal -> Diode_THT:D_DO-35_SOD27_P10.16mm_Horizontal
Changed lines of the file:
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@@
 			)
 		)
-		(property "Footprint" "Capacitor_THT:CP_Radial_D5.0mm_P2.50mm"
+		(property "Footprint" "Capacitor_THT:CP_Radial_D5.0mm_P2.00mm"
 			(at 187.96 102.87 0)
 			(effects
@@
 			)
 		)
-		(property "Footprint" "Diode_THT:D_A-405_P10.16mm_Horizontal"
+		(property "Footprint" "Diode_THT:D_DO-35_SOD27_P10.16mm_Horizontal"
 			(at 177.8 96.52 0)
 			(effects

Commit message: Update schematic values and add backup
Modify several component values in SMEE-DESIGNPROJECT.kicad_sch to new expected values (1k -> 470, 220k -> 2.2k, 65 -> 150, 55 -> 140, 10p -> 470p). Add a timestamped project backup ZIP (SMEE-DESIGNPROJECT-2026-03-19_125239.zip) and a KiCad lock file (~SMEE-DESIGNPROJECT.kicad_sch.lck) containing hostname/username. These changes update circuit component values and include a saved backup/lock for the editing session.
Parts:
- C1: value 10p -> 470p
- R1: value 65 -> 150
- R2: value 55 -> 140
- R4: value 1k -> 470
- R5: value 220k -> 2.2k
Changed lines of the file:
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@@
 			)
 		)
-		(property "Value" "1k"
+		(property "Value" "470"
 			(at 93.98 96.5199 0)
 			(effects
@@
 			)
 		)
-		(property "Value" "220k"
+		(property "Value" "2.2k"
 			(at 93.98 109.2199 0)
 			(effects
@@
 			)
 		)
-		(property "Value" "65"
+		(property "Value" "150"
 			(at 158.75 60.706 90)
 			(effects
@@
 			)
 		)
-		(property "Value" "55"
+		(property "Value" "140"
 			(at 158.75 68.58 90)
 			(effects
@@
 			)
 		)
-		(property "Value" "10p"
+		(property "Value" "470p"
 			(at 95.25 121.9199 0)
 			(effects
